File: KiCAD PCB/PCB_Completo/PCB_Completo.kicad_sch (KiCad schematic)
At the start: 9 parts, among them U1 LM317L_SOT-89, U2 LM337_TO3

Commit message: Actualización y corrección de errores
Parts:
- removed R1, R2, R3, R4: R, symbol Device:R
- removed RV1: R_Potentiometer, symbol Device:R_Potentiometer
- removed U1: LM317L_SOT-89, Package_TO_SOT_SMD:SOT-89-3, symbol Regulator_Linear:LM317L_SOT-89
- added 14.5k1: RCH, symbol Device:R_Potentiometer_Trim
- added 15k1: RCC, symbol Device:R_Potentiometer_Trim
- added 18k1: RS, symbol Device:R_Potentiometer_Trim
- added 4.7M1: RL, symbol Device:R_Potentiometer_Trim
- added C3, C5, C7: 0.1uF, symbol Device:C
- added C4, C6, C8, CL1: 1uF, symbol Device:C
- added J1, J2: Conn_01x02, symbol Connector_Generic:Conn_01x02
- added R11, R7, R8: 120, symbol Device:R
- added R5: 744, symbol Device:R
- added R9: 1032, symbol Device:R
- added RV2: 1032, symbol Device:R_Potentiometer
- added SW1: SW_DPST_x2, symbol Switch:SW_DPST_x2
- added TH1: Thermistor, symbol Device:Thermistor
- added U1: LM350_TO3, Package_TO_SOT_THT:TO-3, symbol Regulator_Linear:LM350_TO3
- added U4: LM337_TO3, Package_TO_SOT_THT:TO-3, symbol Regulator_Linear:LM337_TO3
Connections:
- net at Hy1.1: now also 14.5k1.2, 15k1.2, 18k1.2
- net GND: now reaches Hy1.10 (VS)
- net GND: now also Hy1.11 (GND), Hy1.12 (GND), Hy1.8 (VDD), Hy2.1, Hy2.17, Hy2.18, Hy2.19, Hy2.20, C3.2, C4.1, C4.2, C5.2, C6.2, C7.2, C8.2, J1.2 (Pin_2), R5.2, R7.2, R9.1, RV2.2, U1.3 (VO)
- net TEC_H: now reaches Hy1.13 (TEC_H+)
- net TEC_H: now also J2.1 (Pin_1)
- net at Hy1.2: now also 14.5k1.3
- net at Hy1.3: now also 15k1.3, CL1.1
- net at Hy1.5: now also 4.7M1.3
- net at Hy1.6: now also TH1.1
- net at Hy1.7: now also 18k1.3, TH1.2
- net TEC_C: now reaches Hy1.9 (TEC_C-)
- net TEC_C: now also J2.2 (Pin_2)
- net at U2.1 (ADJ): now also R8.1, R9.2
- net VEE: now reaches U2.2 (VO)
- net VEE: now also Hy2.10, Hy2.11, Hy2.16, Hy2.9, C6.1, R8.2, SW1.1 (A)
- net -15V: now reaches U2.3 (VI)
- net -15V: now also C5.1, C7.1, U4.3 (VI)
- net at Hy2.12: now also J1.1 (Pin_1)
- net VMOD: now reaches Hy2.21
- net VMOD: now also C8.1, R11.2, U4.2 (VO)
- net at Hy2.7: now also SW1.2 (B)
- new net: 4.7M1.2, CL1.2
- new net: R11.1, RV2.1, U4.1 (ADJ)
- new net: R5.1, R7.1, U1.1 (ADJ)
- new net +15V: C3.1, U1.2 (VI)
- no-connect marks 0 -> 6
Other:
- note added: "Circuito de alimentación negativa"
- note added: "Circuito de alimentación positiva"
- note added: "Configuración control de corriente Hy6340"
- note added: "Control de corriente y temperatura para diodos laser de alta corriente"
- note added: "Control de temperatura Hy5640"
- note added: "RS 18k => T = 10°C ICmax = 1A => RCC = 15k IHmax = 0.7*ICmax = 0.7(1A) => RCH = 14.5k RL = 4.7M y CL = 1uF => RC = 5s"
- note added: "VEE = 9V"
- note added: "VMOD = -9V si RVAR = 744 VMOD = -12V si RVAR = 1032"
- moved on the sheet: Hy1, Hy2, U2

Commit message: Se agrega el PCB completo
Parts:
- removed SW1: SW_DPST_x2, symbol Switch:SW_DPST_x2
- removed U1: LM350_TO3, Package_TO_SOT_THT:TO-3, symbol Regulator_Linear:LM350_TO3
- removed U2, U4: LM337_TO3, Package_TO_SOT_THT:TO-3, symbol Regulator_Linear:LM337_TO3
- added J1, J2, J5: Conn_01x02, Connector:JWT_A3963_1x02_P3.96mm_Vertical, symbol Connector_Generic:Conn_01x02
- added R6: 15k, Resistor_THT:R_Axial_DIN0207_L6.3mm_D2.5mm_P15.24mm_Horizontal, symbol Device:R
- added R7: 3k, Resistor_THT:R_Axial_DIN0207_L6.3mm_D2.5mm_P15.24mm_Horizontal, symbol Device:R
- added SW2: SW_DIP_x01, Button_Switch_THT:SW_DIP_SPSTx01_Slide_6.7x4.1mm_W7.62mm_P2.54mm_LowProfile, symbol Switch:SW_DIP_x01
- added U1, U2: LM337T, TerminalBlock_Philmore:TerminalBlock_Philmore_TB133_1x03_P5.00mm_Horizontal, symbol LM337T:LM337T
- added U4: LM350T, TerminalBlock_MetzConnect:TerminalBlock_MetzConnect_Type094_RT03503HBLU_1x03_P5.00mm_Horizontal, symbol LM350T:LM350T
- C1: renamed from C3; footprint (none) -> Capacitor_THT:C_Axial_L3.8mm_D2.6mm_P7.50mm_Horizontal
- C2: renamed from C5; footprint (none) -> Capacitor_THT:C_Axial_L3.8mm_D2.6mm_P7.50mm_Horizontal
- C3: renamed from C7; footprint (none) -> Capacitor_THT:C_Axial_L3.8mm_D2.6mm_P7.50mm_Horizontal
- C4: renamed from C6; footprint (none) -> Capacitor_THT:C_Axial_L3.8mm_D2.6mm_P7.50mm_Horizontal
- C5: renamed from C8; footprint (none) -> Capacitor_THT:C_Axial_L3.8mm_D2.6mm_P7.50mm_Horizontal
- C6: renamed from C4; footprint (none) -> Capacitor_THT:C_Axial_L3.8mm_D2.6mm_P7.50mm_Horizontal
- CL1: footprint (none) -> Capacitor_THT:C_Axial_L3.8mm_D2.6mm_P7.50mm_Horizontal
- Hy1: renamed from Hy2; footprint (none) -> Hytek_Controllers:Hy6340
- Hy2: renamed from Hy1; footprint (none) -> Hytek_Controllers:Hy5640
- J3: renamed from J1; footprint (none) -> Connector:JWT_A3963_1x02_P3.96mm_Vertical
- J4: renamed from J2; footprint (none) -> Connector:JWT_A3963_1x02_P3.96mm_Vertical
- R1: renamed from R5; footprint (none) -> Resistor_THT:R_Axial_DIN0207_L6.3mm_D2.5mm_P15.24mm_Horizontal
- R2: renamed from R9; footprint (none) -> Resistor_THT:R_Axial_DIN0207_L6.3mm_D2.5mm_P15.24mm_Horizontal
- R3: renamed from R7; footprint (none) -> Resistor_THT:R_Axial_DIN0207_L6.3mm_D2.5mm_P15.24mm_Horizontal
- R4: renamed from R8; footprint (none) -> Resistor_THT:R_Axial_DIN0207_L6.3mm_D2.5mm_P15.24mm_Horizontal
- R5: renamed from R11; footprint (none) -> Resistor_THT:R_Axial_DIN0207_L6.3mm_D2.5mm_P15.24mm_Horizontal
- RCC1: renamed from 15k1; value RCC -> 15k1; footprint (none) -> Potentiometer_THT:Potentiometer_Bourns_3296W_Vertical
- RCH1: renamed from 14.5k1; value RCH -> 14.5k1; footprint (none) -> Potentiometer_THT:Potentiometer_Bourns_3296W_Vertical
- RL1: renamed from 4.7M1; value RL -> 4.7M1; footprint (none) -> Potentiometer_THT:Potentiometer_Bourns_3296W_Vertical
- RS1: renamed from 18k1; value RS -> 18k1; footprint (none) -> Potentiometer_THT:Potentiometer_Bourns_3296W_Vertical
- RV1: renamed from RV2; footprint (none) -> Potentiometer_THT:Potentiometer_Bourns_3296W_Vertical
- TH1: footprint (none) -> Resistor_SMD:R_0805_2012Metric_Pad1.20x1.40mm_HandSolder
Connections:
- net +15V: now also J1.1 (Pin_1), U4.3 (VIN)
- net -15V: now also J2.1 (Pin_1), U1.2 (IN), U2.2 (IN)
- net GND: now also R1.1, R2.2, J1.2 (Pin_2), J2.2 (Pin_2), R6.2; no longer C6.1, Hy2.10 (VS), Hy2.8 (VDD), R1.2, R2.1, R3.2
- net VEE: now also SW2.1, U1.3 (OUT)
- net VMOD: now also U2.3 (OUT)
- net at R5.1, RV1.1: now also U2.1 (ADJ)
- net at R3.1: now also R1.2, U4.1 (ADJ); no longer R1.1
- net at R4.1: now also R2.1, U1.1 (ADJ); no longer R2.2
- net at Hy1.7: now also SW2.2
- net at Hy1.8: now also J5.1 (Pin_1), R7.1
- new net: J5.2 (Pin_2), R6.1, R7.2
- new net VDD: C6.1, Hy2.10 (VS), Hy2.8 (VDD), R3.2, U4.2 (VOUT)
- no-connect marks 6 -> 5
Other:
- note added: "Pinouts arduino"
- moved on the sheet: C1, C2, C3, C4, C5, Hy1, J3, R1, R2, R3, R4, R5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
